Commit message: 正式提交：找回丢失的编译配置文件并清理冗余

File: rl_sar_12-27/src/robots/go2_description/urdf/_d435.urdf.xacro (robot description, xacro)
@@ -53,16 +53,4 @@
         <material name="${name}_aluminum"/>
       </visual>
-      <collision>
-        <origin xyz="0 ${-d435_cam_depth_py} 0" rpy="0 0 0"/>
-        <geometry>
-        <box size="${d435_cam_depth} ${d435_cam_width} ${d435_cam_height}"/>
-        </geometry>
-      </collision>
-      <inertial>
-        <!-- The following are not reliable values, and should not be used for modeling -->
-        <mass value="0.564" />
-        <origin xyz="0 0 0" />
-        <inertia ixx="0.003881243" ixy="0.0" ixz="0.0" iyy="0.000498940" iyz="0.0" izz="0.003879257" />
-      </inertial>
     </link>
     <!-- camera depth joints and links -->

File: rl_sar_12-27/src/robots/go2_description/urdf/go2_description-c.urdf (robot description, URDF)
Before this commit: robot go2_description, 30 links, 29 joints
Links:
- link radar: mass 0 -> None

File: rl_sar_12-27/src/robots/go2_description/urdf/go2_description.urdf (robot description, URDF)
Before this commit: robot go2_description, 30 links, 29 joints
Links:
- link radar: mass 0 -> None

File: rl_sar_12-27/src/robots/go2_description/xacro/gazebo.xacro (robot description, xacro)
@@ -157,4 +157,48 @@
         <origin xyz="0.32 0 0.07" rpy="0 0.35 0"/>
     </xacro:sensor_d435>
+    <!-- MID360-style lidar for FAST-LIVO2 simulation.
+         It publishes PointCloud2 on /livox/lidar with Gazebo sim time. -->
+    <gazebo reference="radar">
+      <sensor name="mid360_lidar" type="gpu_ray">
+        <always_on>true</always_on>
+        <visualize>false</visualize>
+        <update_rate>10</update_rate>
+        <pose>0 0 0 0 0 0</pose>
+        <ray>
+          <scan>
+            <horizontal>
+              <samples>1024</samples>
+              <resolution>1</resolution>
+              <min_angle>-3.141592653589793</min_angle>
+              <max_angle>3.141592653589793</max_angle>
+            </horizontal>
+            <vertical>
+              <samples>64</samples>
+              <resolution>1</resolution>
+              <min_angle>-0.126012</min_angle>
+              <max_angle>0.963771</max_angle>
+            </vertical>
+          </scan>
+          <range>
+            <min>0.1</min>
+            <max>70.0</max>
+            <resolution>0.01</resolution>
+          </range>
+          <noise>
+            <type>gaussian</type>
+            <mean>0.0</mean>
+            <stddev>0.01</stddev>
+          </noise>
+        </ray>
+        <plugin name="mid360_lidar_controller" filename="libgazebo_ros_ray_sensor.so">
+          <ros>
+            <namespace>/</namespace>
+            <remapping>~/out:=/livox/lidar</remapping>
+          </ros>
+          <output_type>sensor_msgs/PointCloud2</output_type>
+          <frame_name>radar</frame_name>
+        </plugin>
+      </sensor>
+    </gazebo>
     <gazebo reference="imu_link">
       <sensor name="imu_sensor" type="imu">
@@ -162,6 +206,7 @@
           <ros>
             <namespace>/</namespace>
-            <remapping>~/out:=imu</remapping>
+            <remapping>~/out:=/imu</remapping>
           </ros>
+          <frame_name>imu_link</frame_name>
           <initial_orientation_as_reference>false</initial_orientation_as_reference>
         </plugin>
